File: kicad-level/level.kicad_pcb (KiCad board)
At the start: 2 copper layers, 37.7 x 27.7 mm, 6 parts, among them J1 Conn_01x01_Pin, J2 Conn_01x08_Pin, J3 Conn_01x01_Pin, U1 ULN2803A_C845537

Commit message: ajout remerciement pcbway
Parts:
- moved J2 2.84 mm to (186.9, 108.0)
Routing:
- net Net-(J2-Pin_5): track 6.59 -> 4.09 mm
- net Net-(J2-Pin_7): track 7.64 -> 5.14 mm
- net Net-(J2-Pin_6): track 7.11 -> 4.62 mm
- net Net-(J2-Pin_4): track 6.59 -> 4.51 mm
- net Net-(J2-Pin_2): track 7.64 -> 5.56 mm
- net Net-(J2-Pin_3): track 7.11 -> 5.04 mm
- net Net-(J2-Pin_8): track 8.17 -> 6.12 mm
- net Net-(J2-Pin_1): track 8.17 -> 6.63 mm
Other:
- board size 37.7 x 27.7 mm -> 34.3 x 27.9 mm
Changed lines of the file:
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@@
 			(outputformat 1)
 			(mirror no)
-			(drillshape 1)
+			(drillshape 0)
 			(scaleselection 1)
-			(outputdirectory "")
+			(outputdirectory "pcbway/")
 		)
 	)
@@
 	(footprint "Connector_PinHeader_2.54mm:PinHeader_1x08_P2.54mm_Vertical"
 		(layer "F.Cu")
-		(at 189.75 107.53 180)
+		(at 186.944 107.95 180)
 		(descr "Through hole straight pin header, 1x08, 2.54mm pitch, single row")
 		(tags "Through hole pin header THT 1x08 2.54mm single row")
@@
 	)
 	(gr_rect
-		(start 154.94 85.598)
-		(end 192.659 113.284)
+		(start 154.94 85.344)
+		(end 189.23 113.284)
 		(stroke
 			(width 0.05)
@@
 	)
 	(gr_text "gnd"
-		(at 179.832 89.916 0)
+		(at 170.688 89.916 0)
 		(layer "F.SilkS")
 		(effects
 			(font
-				(size 3 3)
+				(size 2 2)
 				(thickness 0.5)
 				(bold yes)
@@
 	)
 	(gr_text "5v"
-		(at 180.34 110.49 0)
+		(at 180.848 111.252 0)
 		(layer "F.SilkS")
 		(effects
 			(font
-				(size 3 3)
+				(size 2 2)
 				(thickness 0.5)
 				(bold yes)
@@
 	)
 	(segment
+		(start 186.944 107.036)
+		(end 186.944 107.95)
+		(width 0.2)
+		(layer "F.Cu")
+		(net 18)
+	)
+	(segment
 		(start 182.905 102.997)
-		(end 184.785 102.997)
-		(width 0.5)
+		(end 186.944 107.036)
+		(width 0.2)
 		(layer "F.Cu")
 		(net 18)
 	)
 	(segment
-		(start 184.785 102.997)
-		(end 189.23 107.442)
-		(width 0.5)
-		(layer "F.Cu")
-		(net 18)
-	)
-	(segment
-		(start 186.055 101.727)
-		(end 189.23 104.902)
-		(width 0.5)
+		(start 182.905 101.727)
+		(end 183.261 101.727)
+		(width 0.2)
 		(layer "F.Cu")
 		(net 19)
 	)
 	(segment
-		(start 182.905 101.727)
-		(end 186.055 101.727)
-		(width 0.5)
+		(start 183.261 101.727)
+		(end 186.944 105.41)
+		(width 0.2)
 		(layer "F.Cu")
 		(net 19)
@@
 	(segment
 		(start 182.905 100.457)
-		(end 187.325 100.457)
-		(width 0.5)
+		(end 184.531 100.457)
+		(width 0.2)
 		(layer "F.Cu")
 		(net 20)
 	)
 	(segment
-		(start 187.325 100.457)
-		(end 189.23 102.362)
-		(width 0.5)
+		(start 184.531 100.457)
+		(end 186.944 102.87)
+		(width 0.2)
 		(layer "F.Cu")
 		(net 20)
 	)
 	(segment
+		(start 185.801 99.187)
+		(end 186.944 100.33)
+		(width 0.2)
+		(layer "F.Cu")
+		(net 21)
+	)
+	(segment
 		(start 182.905 99.187)
-		(end 188.595 99.187)
-		(width 0.5)
+		(end 185.801 99.187)
+		(width 0.2)
 		(layer "F.Cu")
 		(net 21)
 	)
 	(segment
-		(start 188.595 99.187)
-		(end 189.23 99.822)
-		(width 0.5)
-		(layer "F.Cu")
-		(net 21)
-	)
-	(segment
-		(start 188.595 97.917)
-		(end 189.23 97.282)
-		(width 0.5)
+		(start 182.905 97.917)
+		(end 186.817 97.917)
+		(width 0.2)
 		(layer "F.Cu")
 		(net 22)
 	)
 	(segment
-		(start 182.905 97.917)
-		(end 188.595 97.917)
-		(width 0.5)
+		(start 186.817 97.917)
+		(end 186.944 97.79)
+		(width 0.2)
 		(layer "F.Cu")
 		(net 22)
@@
 	(segment
 		(start 182.905 96.647)
-		(end 187.325 96.647)
-		(width 0.5)
+		(end 185.547 96.647)
+		(width 0.2)
 		(layer "F.Cu")
 		(net 23)
 	)
 	(segment
-		(start 187.325 96.647)
-		(end 189.23 94.742)
-		(width 0.5)
+		(start 185.547 96.647)
+		(end 186.944 95.25)
+		(width 0.2)
 		(layer "F.Cu")
 		(net 23)
 	)
 	(segment
+		(start 184.277 95.377)
+		(end 186.944 92.71)
+		(width 0.2)
+		(layer "F.Cu")
+		(net 24)
+	)
+	(segment
 		(start 182.905 95.377)
-		(end 186.055 95.377)
-		(width 0.5)
+		(end 184.277 95.377)
+		(width 0.2)
 		(layer "F.Cu")
 		(net 24)
 	)
 	(segment
-		(start 186.055 95.377)
-		(end 189.23 92.202)
-		(width 0.5)
-		(layer "F.Cu")
-		(net 24)
+		(start 186.944 90.942999)
+		(end 186.944 90.17)
+		(width 0.2)
+		(layer "F.Cu")
+		(net 25)
 	)
 	(segment
 		(start 182.905 94.107)
-		(end 184.785 94.107)
-		(width 0.5)
+		(end 183.779999 94.107)
+		(width 0.2)
 		(layer "F.Cu")
 		(net 25)
 	)
 	(segment
-		(start 184.785 94.107)
-		(end 189.23 89.662)
-		(width 0.5)
+		(start 183.779999 94.107)
+		(end 186.944 90.942999)
+		(width 0.2)
 		(layer "F.Cu")
 		(net 25)
