File: kicad-level/level.kicad_sch (KiCad schematic)
At the start: 6 parts, among them J1 Conn_01x01_Pin, J2 Conn_01x08_Pin, J3 Conn_01x01_Pin, U1 ULN2803A_C845537

Commit message: misa a jour pcb plus petit
Connections:
- net GND: no longer U1.10 (COM)
Changed lines of the file:
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@@
 	(paper "A4")
-	(junction
-		(at 167.64 127)
-		(diameter 0)
-		(color 0 0 0 0)
-	)
 	(junction
 		(at 154.94 127)
@@
 		)
 		(stroke
-			(width 0)
-			(type default)
-		)
-	)
-	(wire
-		(pts
-			(xy 167.64 90.17) (xy 167.64 127)
-		)
-		(stroke
-			(width 0)
-			(type default)
-		)
-	)
-	(wire
-		(pts
-			(xy 165.1 90.17) (xy 167.64 90.17)
-		)
-		(stroke
